File: piccolo.kicad_pcb (KiCad board)
At the start: 2 copper layers, 21 x 51 mm, 42 parts, among them J0 CON_PICO_40W, J1 USB_C_Receptacle_USB2.0, J2 Debug, Q1 DMG1012T, SW1 BOOTSEL, U1 RP2040, U2 ME6217C33M5, U3 MX25R1635FZUIL0, X1 SIT1602AI-22-33E-12.000000D

Commit message: Initial PCB design
Parts:
- added C16: 100n 6.3V, Capacitor_SMD:C_0201_0603Metric, F.Cu at (118.9, 77.4)
- added D3: Yellow, LED_SMD:LED_0603_1608Metric, F.Cu at (116.8, 50.5)
- C3: footprint Capacitor_SMD:C_0201_0603Metric -> Capacitor_SMD:C_0402_1005Metric
- R8: value 100k -> 470R
- U1: footprint Package_DFN_QFN:QFN-56-1EP_7x7mm_P0.4mm_EP5.6x5.6mm -> agausmann:RP2040_QFN-56-1EP_7x7mm_P0.4mm_EP3.2x3.2mm_ThermalVias
- moved C15 7.65 mm to (117.9, 59.5), turned to 0 degrees
- moved R13 5.85 mm to (123.2, 62.9)
- moved R12 5.74 mm to (122.4, 62.9)
- moved C11 4.96 mm to (121.0, 62.9)
- moved R11 4.95 mm to (119.1, 57.7), turned to 0 degrees
- moved C10 4.94 mm to (121.7, 62.9)
- moved R10 4.91 mm to (127.7, 67.3)
- moved R1 4.67 mm to (127.7, 68.3)
- moved C18 4.45 mm to (118.1, 58.7)
- moved R5 3.93 mm to (128.3, 55.9), turned to -90 degrees
- moved C7 3.77 mm to (126.5, 65.3)
- moved C6 3.40 mm to (126.4, 69.3)
- moved U3 3.23 mm to (118.6, 61.8), turned to 90 degrees
- moved R3 3.20 mm to (119.4, 49.7), turned to 180 degrees
- moved C12 3.13 mm to (124.0, 62.7)
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Connections:
- net /USB_DM renamed /USB_D-
- net /USB_DP renamed /USB_D+
- J0 pad 33: GNDA -> GND
- R8 pad 2: GND -> Net-(R8-Pad2)
Routing:
- net GND: track 0.00 -> 87.0 mm, vias 0 -> 24
- net +3V3: track 0.00 -> 41.6 mm, vias 0 -> 4
- net /GPIO0: track 0.00 -> 27.3 mm
- net VBUS: track 0.00 -> 26.4 mm, vias 0 -> 4
- net /GPIO1: track 0.00 -> 25.2 mm
- net /GPIO25: track 0.00 -> 23.4 mm, vias 0 -> 2
- net /GPIO23: track 0.00 -> 23.2 mm, vias 0 -> 2
- net /GPIO15: track 0.00 -> 23.0 mm
- net /GPIO16: track 0.00 -> 22.2 mm
- net /SWCLK: track 0.00 -> 21.9 mm
- net /GPIO2: track 0.00 -> 20.5 mm
- net /GPIO14: track 0.00 -> 20.3 mm
- net /GPIO17: track 0.00 -> 19.2 mm
- net /SWDIO: track 0.00 -> 18.6 mm
- net /GPIO3: track 0.00 -> 18.4 mm
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- added copper zone on F.Cu, net +1V1
- added copper zone on F.Cu, net +3V3
- added copper zone on F.Cu, net /USB_D+
- added copper zone on F.Cu, net /USB_D-
- added copper zone on F.Cu, net /VSYS
- added copper zone on B.Cu, net GND
- added copper zone on F.Cu, net GND
- added copper zone on F.Cu, net VBUS
Other:
- board text added: "3V3"
- board text added: "3V3_EN"
- board text added: "ADC_VREF"
- board text added: "Adam Gausmann"
- board text added: "BOOTSEL"
- board text added: "DEBUG"
- board text added: "GND"
- board text added: "GP0"
- board text added: "GP1"
- board text added: "GP10"
- board text added: "GP11"
- board text added: "GP12"
- board text added: "GP13"
- board text added: "GP14"
- board text added: "GP15"
- board text added: "GP16"
- board text added: "GP17"
- board text added: "GP18"
- board text added: "GP19"
- board text added: "GP2"
- board text added: "GP20"
- board text added: "GP21"
- board text added: "GP22"
- board text added: "GP26_A0"
- board text added: "GP27_A1"
- board text added: "GP28_A2"
- board text added: "GP3"
- board text added: "GP4"
- board text added: "GP5"
- board text added: "GP6"
- board text added: "GP7"
- board text added: "GP8"
- board text added: "GP9"
- board text added: "PICCOLO"
- board text added: "RUN"
- board text added: "RevXX"
- board text added: "SWCLK"
- board text added: "SWDIO"
- board text added: "USB"
- board text added: "VBUS"
- board text added: "VSYS"
- board text added: "YYYY-MM-DD"
