File: piccolo.kicad_sch (KiCad schematic)
At the start: 0 parts

Commit message: Port schematic and very roughly position components
Parts:
- added C1, C2: 10u 6.3V, Capacitor_SMD:C_0805_2012Metric, symbol Device:C_Small
- added C10, C11, C15, C4, C5, C6, C7, C8, C9: 100n 6.3V, Capacitor_SMD:C_0201_0603Metric, symbol Device:C_Small
- added C12, C13, C14, C18: 2.2u 6.3V, Capacitor_SMD:C_0402_1005Metric, symbol Device:C_Small
- added C3: 1n 25V, Capacitor_SMD:C_0201_0603Metric, symbol Device:C
- added D1: MBR120VLSFT1G, Diode_SMD:D_SOD-123F, symbol Device:D_Schottky
- added D2: Green, LED_SMD:LED_0603_1608Metric, symbol Device:LED
- added J0: CON_PICO_40W, agausmann:RaspberryPi_Pico_OutlineAndPads, symbol Connector_Generic:Conn_02x20_Counter_Clockwise
- added J1: USB_C_Receptacle_USB2.0, Connector_USB:USB_C_Receptacle_HRO_TYPE-C-31-M-12, symbol Connector:USB_C_Receptacle_USB2.0
- added J2: Debug, Connector_PinHeader_2.54mm:PinHeader_1x03_P2.54mm_Vertical, symbol Connector_Generic:Conn_01x03
- added Q1: DMG1012T, Package_TO_SOT_SMD:SOT-523, symbol Device:Q_NMOS_GSD
- added R1: 10k, Resistor_SMD:R_0402_1005Metric, symbol Device:R
- added R10: 5.6k, Resistor_SMD:R_0402_1005Metric, symbol Device:R
- added R11: 1k, Resistor_SMD:R_0402_1005Metric, symbol Device:R_Small
- added R12, R13: 27R, Resistor_SMD:R_0201_0603Metric, symbol Device:R_Small
- added R16, R17: 5.1k, Resistor_SMD:R_0402_1005Metric, symbol Device:R_Small
- added R2: 100k, Resistor_SMD:R_0402_1005Metric, symbol Device:R_Small
- added R3: 470R, Resistor_SMD:R_0402_1005Metric, symbol Device:R_Small
- added R4: NO-FIT, Resistor_SMD:R_0402_1005Metric, symbol Device:R_Small
- added R5: 200k, Resistor_SMD:R_0402_1005Metric, symbol Device:R
- added R6, R8: 100k, Resistor_SMD:R_0402_1005Metric, symbol Device:R
- added R7: 200R, Resistor_SMD:R_0603_1608Metric, symbol Device:R_Small
- added R9: 1R, Resistor_SMD:R_0402_1005Metric, symbol Device:R_Small
- added SW1: BOOTSEL, Button_Switch_SMD:SW_Push_1P1T_NO_Vertical_Wuerth_434133025816, symbol Switch:SW_Push
- added U1: RP2040, Package_DFN_QFN:QFN-56-1EP_7x7mm_P0.4mm_EP5.6x5.6mm, symbol agausmann:RP2040
- added U2: ME6217C33M5, Package_TO_SOT_SMD:SOT-23-5, symbol agausmann:ME6217C33M5
- added U3: MX25R1635FZUIL0, agausmann:USON-8-1EP_3x2mm_P0.5mm_EP0.2x1.6mm, symbol Memory_Flash:W25Q32JVZP
- added X1: SIT1602AI-22-33E-12.000000D, agausmann:SiT1602xx-2_3.2x2.5mm, symbol agausmann:SIT1602
Connections:
- new net: C3.1, Q1.3 (D), R5.2, R6.1
- new net: R11.2, SW1.2
- new net: J1.B5 (CC2), R16.2
- new net: R13.2, U1.46 (USB_DM)
- new net: D2.2 (A), R3.2
- new net: J1.A5 (CC1), R17.1
- new net: R12.2, U1.47 (USB_DP)
- new net +1V1: C11.1, C12.1, C9.1, U1.23 (DVDD), U1.45 (VREG_VOUT), U1.50 (DVDD)
- new net +3V3: C10.1, C14.1, C15.1, C18.1, C2.1, C4.1, C5.1, C6.1, C7.1, C8.1, J0.36 (Pin_36), Q1.1 (G), R4.1, R7.1, U1.1 (IOVDD), U1.10 (IOVDD), U1.22 (IOVDD), U1.33 (IOVDD), U1.42 (IOVDD), U1.44 (VREG_VIN), U1.48 (USB_VDD), U1.49 (IOVDD), U2.5 (OUT), U3.8 (VCC), X1.1 (OE), X1.4 (VDD)
- new net 3V3_EN: J0.37 (Pin_37), R2.1, U2.3 (EN)
- new net ADC_AVDD: C13.1, R9.2, U1.43 (ADC_AVDD)
- new net ADC_VREF: J0.35 (Pin_35), R7.2, R9.1
- new net GND: C1.1, C10.2, C11.2, C12.2, C13.2, C14.2, C15.2, C18.2, C2.2, C3.2, C4.2, C5.2, C6.2, C7.2, C8.2, C9.2, D2.1 (K), J0.13 (Pin_13), J0.18 (Pin_18), J0.23 (Pin_23), J0.28 (Pin_28), J0.3 (Pin_3), J0.38 (Pin_38), J0.8 (Pin_8), J1.A1 (GND), J1.A12 (GND), J1.B1 (GND), J1.B12 (GND), J1.S1 (SHIELD), J2.2 (Pin_2), R1.2, R16.1, R17.2, R6.2, R8.2, SW1.1, U1.19 (TESTEN), U1.57 (GND), U2.2 (GND), U3.4 (GND), X1.2 (GND)
- new net GNDA: J0.33 (Pin_33)
- new net GPIO0: J0.1 (Pin_1), U1.2 (GPIO0)
- new net GPIO1: J0.2 (Pin_2), U1.3 (GPIO1)
- new net GPIO10: J0.14 (Pin_14), U1.13 (GPIO10)
- new net GPIO11: J0.15 (Pin_15), U1.14 (GPIO11)
- new net GPIO12: J0.16 (Pin_16), U1.15 (GPIO12)
- new net GPIO13: J0.17 (Pin_17), U1.16 (GPIO13)
- new net GPIO14: J0.19 (Pin_19), U1.17 (GPIO14)
- new net GPIO15: J0.20 (Pin_20), U1.18 (GPIO15)
- new net GPIO16: J0.21 (Pin_21), U1.27 (GPIO16)
- new net GPIO17: J0.22 (Pin_22), U1.28 (GPIO17)
- new net GPIO18: J0.24 (Pin_24), U1.29 (GPIO18)
- new net GPIO19: J0.25 (Pin_25), U1.30 (GPIO19)
- new net GPIO2: J0.4 (Pin_4), U1.4 (GPIO2)
- new net GPIO20: J0.26 (Pin_26), U1.31 (GPIO20)
- new net GPIO21: J0.27 (Pin_27), U1.32 (GPIO21)
- new net GPIO22: J0.29 (Pin_29), U1.34 (GPIO22)
- new net GPIO23: R8.1, U1.35 (GPIO23)
- new net GPIO24: R1.1, R10.2, U1.36 (GPIO24)
- new net GPIO25: R3.1, U1.37 (GPIO25)
- new net GPIO26_ADC0: J0.31 (Pin_31), U1.38 (GPIO26/ADC0)
- new net GPIO27_ADC1: J0.32 (Pin_32), U1.39 (GPIO27/ADC1)
- new net GPIO28_ADC2: J0.34 (Pin_34), U1.40 (GPIO28/ADC2)
- new net GPIO29_ADC3: Q1.2 (S), U1.41 (GPIO29/ADC3)
- new net GPIO3: J0.5 (Pin_5), U1.5 (GPIO3)
- new net GPIO4: J0.6 (Pin_6), U1.6 (GPIO4)
- new net GPIO5: J0.7 (Pin_7), U1.7 (GPIO5)
- new net GPIO6: J0.9 (Pin_9), U1.8 (GPIO6)
- new net GPIO7: J0.10 (Pin_10), U1.9 (GPIO7)
- new net GPIO8: J0.11 (Pin_11), U1.11 (GPIO8)
- new net GPIO9: J0.12 (Pin_12), U1.12 (GPIO9)
- new net QSPI_SCLK: U1.52 (QSPI_SCLK), U3.6 (CLK)
- new net QSPI_SD0: U1.53 (QSPI_SD0), U3.5 (DI(IO0))
- new net QSPI_SD1: U1.55 (QSPI_SD1), U3.2 (DO(IO1))
- new net QSPI_SD2: U1.54 (QSPI_SD2), U3.3 (IO2)
- new net QSPI_SD3: U1.51 (QSPI_SD3), U3.7 (IO3)
- new net QSPI_SS: R11.1, R4.2, U1.56 (QSPI_SS_N), U3.1 (~{CS})
- new net RUN: J0.30 (Pin_30), U1.26 (RUN)
- new net SWCLK: J2.1 (Pin_1), U1.24 (SWCLK)
- new net SWDIO: J2.3 (Pin_3), U1.25 (SWDIO)
- new net USB_DM: J1.A7 (D-), J1.B7 (D-), R13.1
- new net USB_DP: J1.A6 (D+), J1.B6 (D+), R12.1
- new net VBUS: D1.2 (A), J0.40 (Pin_40), J1.A4 (VBUS), J1.A9 (VBUS), J1.B4 (VBUS), J1.B9 (VBUS), R10.1
- new net VSYS: C1.2, D1.1 (K), J0.39 (Pin_39), R2.2, R5.1, U2.1 (IN)
- new net XIN: U1.20 (XIN), X1.3 (OUT)
- no-connect marks 0 -> 4
Other:
- note added: "NOTE - Max clock rate is 80MHz System clock may have to be reduced to stay within spec for this chip."
- note added: "No PS feature"
- note added: "Prefer MEMS oscillators over crystals"
- note added: "Replaced Micro-USB with USB-C"
- note added: "Replaced buck-boost with LDO regulator."
- note added: "Software VBUS detect"

Commit message: Initial PCB design
Parts:
- removed R8: 100k, Resistor_SMD:R_0402_1005Metric, symbol Device:R
- added C16: 100n 6.3V, Capacitor_SMD:C_0201_0603Metric, symbol Device:C_Small
- added D3: Yellow, LED_SMD:LED_0603_1608Metric, symbol Device:LED
- added R8: 470R, Resistor_SMD:R_0402_1005Metric, symbol Device:R_Small
- C1, C2: LCSC (none) -> C440198
- C10, C11, C15, C4, C5, C6, C7, C8, C9: LCSC (none) -> C160831
- C12, C13, C14, C18: LCSC (none) -> C12530
- C3: footprint Capacitor_SMD:C_0201_0603Metric -> Capacitor_SMD:C_0402_1005Metric; LCSC (none) -> C66942
- D1: LCSC (none) -> C123070
- D2: LCSC (none) -> C72043
- R1: LCSC (none) -> C25744
- R10: LCSC (none) -> C25908
- R11: LCSC (none) -> C11702
- R12, R13: LCSC (none) -> C25100
- R16, R17: LCSC (none) -> C25905
- R2, R6: LCSC (none) -> C25741
- R3: LCSC (none) -> C25117
- R5: LCSC (none) -> C25764
- R7: LCSC (none) -> C25087
- R9: LCSC (none) -> C25086
- U1: footprint Package_DFN_QFN:QFN-56-1EP_7x7mm_P0.4mm_EP5.6x5.6mm -> agausmann:RP2040_QFN-56-1EP_7x7mm_P0.4mm_EP3.2x3.2mm_ThermalVias
Connections:
- net GNDA is gone; now on net GND: J0.33 (Pin_33)
- net +3V3: now also C16.1
- net GND: now also C16.2, D3.1 (K)
- net GPIO23: now also R8.1
- net USB_DM renamed USB_D-
- net USB_DP renamed USB_D+
- new net: D3.2 (A), R8.2
Other:
- note added: "Extra pin from regulator not having PS feature - can use it for another indicator"
- note removed: "No PS feature"
- moved on the sheet: D2, R3

Commit message: Fill out BOM
Parts:
- C1, C2: Manufacturer (none) -> Samsung; Part Number (none) -> CL21A106MQFNNNE
- C10, C11, C15, C16, C4, C5, C6, C7, C8, C9: Manufacturer (none) -> Samsung; Part Number (none) -> CL03A104KQ3NNNC
- C12, C13, C14, C18: Manufacturer (none) -> Samsung; Part Number (none) -> CL05A225KQ5NNNC
- C3: Manufacturer (none) -> Kyocera; Part Number (none) -> 04023C102KAT2A
- D1: Manufacturer (none) -> onsemi; Part Number (none) -> MBR120VLSFT1G
- D2: Manufacturer (none) -> Lite-On; Part Number (none) -> LTST-C191KGKT
- D3: value Yellow -> Red; Manufacturer (none) -> Lite-On; Part Number (none) -> LTST-C191KRKT
- J1: Manufacturer (none) -> Korean Hroparts; Part Number (none) -> TYPE-C-31-M-12
- Q1: Manufacturer (none) -> Diodes Inc; Part Number (none) -> DMG1012T
- R1: Manufacturer (none) -> Yageo; Part Number (none) -> RC0402FR-0710KL
- R10: Manufacturer (none) -> Yageo; Part Number (none) -> RC0402FR-075K6L
- R11: Manufacturer (none) -> Yageo; Part Number (none) -> RC0402FR-071KL
- R12, R13: Manufacturer (none) -> Yageo; Part Number (none) -> RC0201FR-0727RL
- R16, R17: Manufacturer (none) -> Yageo; Part Number (none) -> RC0402FR-075K1L
- R2, R6: Manufacturer (none) -> Yageo; Part Number (none) -> RC0402FR-07100KL
- R3, R8: Manufacturer (none) -> Yageo; Part Number (none) -> RC0402FR-07470RL
- R5: Manufacturer (none) -> Yageo; Part Number (none) -> RC0402FR-07200KL
- R7: Manufacturer (none) -> Stackpole; Part Number (none) -> RMCF0603FT200R
- R9: Manufacturer (none) -> Yageo; Part Number (none) -> RC0402FR-071RL
- SW1: Manufacturer (none) -> Wuerth; Part Number (none) -> 434133025816
- U1: Manufacturer (none) -> Raspberry Pi; Part Number (none) -> RP2040
- U2: Manufacturer (none) -> Microne; Part Number (none) -> ME6217C33M5
- U3: value MX25R1635FZUIL0 -> W25Q16JVUXIQ; Manufacturer (none) -> Winbond; Part Number (none) -> W25Q16JVUXIQ
- X1: value SIT1602AI-22-33E-12.000000D -> SIT1602AI-22-33E-12.000000; Manufacturer (none) -> SiTime; Part Number (none) -> SIT1602AI-22-33E-12.000000
